File: translators.kicad_sch (KiCad schematic)
At the start: 26 parts, among them Q2 2N7002, Q3 2N7002, U13 SN74LVC8T245PWR, U14 SN74LVC8T245PWR, U15 SN74LVC1T45DBVR, U16 SN74LVC1T45DBVR, U17 TCA9517ADGKR

Commit message: fix: apply schematic review findings (VIO 5V at power-up, push-pull BOOT, input bias, CC ESD)
Co-Authored-By: Claude Opus 5.5 <noreply@anthropic.com>
Parts:
- removed Q3: 2N7002, Package_TO_SOT_SMD:SOT-23, symbol Transistor_FET:2N7002
- removed R36: 10k, Resistor_SMD:R_0402_1005Metric, symbol Device:R
- removed U13: SN74LVC8T245PWR, Package_SO:TSSOP-24_4.4x7.8mm_P0.65mm, symbol Logic_LevelTranslator:SN74LVC8T245
- removed U15: SN74LVC1T45DBVR, Package_TO_SOT_SMD:SOT-23-6, symbol Logic_LevelTranslator:SN74LVC1T45DBV
- removed U17: TCA9517ADGKR, Package_SO:VSSOP-8_3x3mm_P0.65mm, symbol Logic_LevelTranslator:TCA9517ADGK
- added C53, C54: 100nF/50V, Capacitor_SMD:C_0402_1005Metric, symbol Device:C
- added R45, R46: 100k, Resistor_SMD:R_0402_1005Metric, symbol Device:R
- added R47, R48, R49, R50, R51, R52, R53, R54, R55, R56: 1M, Resistor_SMD:R_0402_1005Metric, symbol Device:R
- added U15: SN74LVC8T245PWR, Package_SO:TSSOP-24_4.4x7.8mm_P0.65mm, symbol Logic_LevelTranslator:SN74LVC8T245
- added U17, U19: SN74LVC1T45DBVR, Package_TO_SOT_SMD:SOT-23-6, symbol Logic_LevelTranslator:SN74LVC1T45DBV
- added U18: TCA9517ADGKR, Package_SO:VSSOP-8_3x3mm_P0.65mm, symbol Logic_LevelTranslator:TCA9517ADGK
- R37, R44: value 100k -> 10k; LCSC C25741 -> C25744; MPN 0402WGF1003TCE -> 0402WGF1002TCE
- R39: value 4.7k -> 100k; LCSC C25900 -> C25741; MPN 0402WGF4701TCE -> 0402WGF1003TCE
- R43: value 100k -> 4.7k; LCSC C25741 -> C25900; MPN 0402WGF1003TCE -> 0402WGF4701TCE
Connections:
- net +3V3: now also R37.2, R43.2, U14.2 (DIR), C53.1, U15.1 (V_{CCA}), U17.1 (VCCA), U18.8 (VCCB), U19.1 (VCCA); no longer R41.2
- net BOOT_DUT_CTL: now also U19.3 (A); no longer R44.1
- net GND: now also R39.2, C53.2, C54.2, R45.2, R46.2, R47.2, R48.2, R49.2, R50.2, R51.2, R52.2, R53.2, U15.11 (GND), U15.12 (GND), U15.13 (GND), U15.14 (B8), U15.2 (DIR), U17.2 (GND), U18.4 (GND), U19.2 (GND); no longer R37.2, R43.2, U14.14 (B8), U14.2 (DIR)
- net I2C_DUT_EN: now also R44.1, U18.5 (EN)
- net I2C_DUT_SCL_MCU: now also R42.1, U18.7 (SCLB); no longer R41.1
- net I2C_DUT_SDA_MCU: now also R43.1, U18.6 (SDAB); no longer R42.1
- net I2C_SCL: now also R40.1, U18.2 (SCLA); no longer R39.1
- net I2C_SDA: now also R41.1, U18.3 (SDAA); no longer R40.1
- net IN1_B: now also R47.1, U15.21 (B1); no longer U14.21 (B1)
- net IN1_MCU: now also U15.3 (A1); no longer U14.3 (A1)
- net IN2_B: now also R48.1, U15.20 (B2); no longer U14.20 (B2)
- net IN2_MCU: now also U15.4 (A2); no longer U14.4 (A2)
- net IN3_B: now also R49.1, U15.19 (B3); no longer U14.19 (B3)
- net IN3_MCU: now also U15.5 (A3); no longer U14.5 (A3)
- net IN4_B: now also R50.1, U15.18 (B4); no longer U14.18 (B4)
- net IN4_MCU: now also U15.6 (A4); no longer U14.6 (A4)
- net LS_OE_N: now also R37.1, U15.22 (~{OE})
- net OUT1_B: now also U14.21 (B1)
- net OUT1_MCU: now also U14.3 (A1)
- net OUT2_B: now also U14.20 (B2)
- net OUT2_MCU: now also U14.4 (A2)
- net OUT3_B: now also U14.19 (B3)
- net OUT3_MCU: now also U14.5 (A3)
- net OUT4_B: now also U14.18 (B4)
- net OUT4_MCU: now also U14.6 (A4)
- net RESET_DUT_CTL: now also R45.1; no longer R43.1
- net SPI_CS_B: now also U14.14 (B8)
- net SPI_CS_MCU: now also U14.10 (A8)
- net SPI_MISO_B: now also R51.1, U15.16 (B6); no longer U14.16 (B6)
- net SPI_MISO_MCU: now also U15.8 (A6); no longer U14.8 (A6)
- net SPI_MOSI_B: now also U14.15 (B7)
- net SPI_MOSI_MCU: now also U14.9 (A7)
- net SPI_SCK_B: now also U14.16 (B6)
- net SPI_SCK_MCU: now also U14.8 (A6)
- net SWCLK_B: now also U16.4 (B), R52.1
- net SWCLK_DIR: now also R38.1, U16.5 (DIR); no longer R37.1
- net SWCLK_MCU: now also U16.3 (A)
- net SWDIO_B: now also R56.1, U17.4 (B); no longer U16.4 (B)
- net SWDIO_DIR: now also R39.1, U17.5 (DIR); no longer R38.1, U16.5 (DIR)
- net SWDIO_MCU: now also U17.3 (A); no longer U16.3 (A)
- net SWO_DUT_B: now also R55.1, U15.15 (B7); no longer U14.15 (B7)
- net SWO_DUT_MCU: now also U15.9 (A7); no longer U14.9 (A7)
- net UART_RX_B: now also R54.1, U15.17 (B5); no longer U14.17 (B5)
- net UART_RX_MCU: now also U15.7 (A5); no longer U14.7 (A5)
- net UART_TX_B: now also U14.17 (B5)
- net UART_TX_MCU: now also U14.7 (A5)
- net VIO: now also R41.2, C54.1, R54.2, R55.2, R56.2, U15.23 (V_{CCB}), U15.24 (V_{CCB}), U17.6 (VCCB), U18.1 (VCCA), U19.6 (VCCB); no longer R39.2
- new net BOOT_B: R53.1, U19.4 (B)
- new net BOOT_DIR: R46.1, U19.5 (DIR)
Other:
- note added: "DUT I2C (A = DUT)"
- note added: "Input bias 1M"
- note added: "Inputs VIO -> 3V3 (DIR = B to A)"
- note added: "Outputs 3V3 -> VIO (DIR = A to B)"
- note added: "RESET (OD) / BOOT (3-state)"
- note added: "SWD probe"
- note removed: "DUT I2C buffer (TCA9517A, A = DUT, B = MCU)"
- note removed: "Inputs DUT -> MCU (SN74LVC8T245, DIR = B to A)"
- note removed: "Outputs MCU -> DUT (SN74LVC8T245, DIR = A to B)"
- note removed: "RESET / BOOT open-drain"
- note removed: "SWD probe (SN74LVC1T45)"

Commit message: fix: apply schematic review (LQFP-80 MCU, fixed-rail EN, VIO from 5V_DUT, buttons, ESD per header)
- STM32G431MBT6 (LQFP-80): 14 more GPIO; BOOT_DIR off PB4 (JTRST pull-up at reset)
- Fixed DUT rails: EN on PE7/PE8 with pull-up (on by default, firmware can cut)
- TPS2116 VIN1 from current-limited 5V_DUT instead of +5V
- Two user push buttons (TS-1187A) on PD0/PD1, BOOT0 solder jumper
- TVS after the PTC, buck Cin 10uF/25V 0805, 5th VDD decoupling cap
- No floating translator inputs (U15 A8 to GND, 1M bias on U14 B side)
- ESD channels grouped per header; datasheet field falls back to LCSC page
- Decoupling capacitors declare the pin they decouple (validated against nets)

Co-Authored-By: Claude Opus 5.5 <noreply@anthropic.com>
Parts:
- removed C43, C44, C45: 100nF/50V, Capacitor_SMD:C_0402_1005Metric, symbol Device:C
- removed R37: 10k, Resistor_SMD:R_0402_1005Metric, symbol Device:R
- removed R38, R39: 100k, Resistor_SMD:R_0402_1005Metric, symbol Device:R
- removed R40: 4.7k, Resistor_SMD:R_0402_1005Metric, symbol Device:R
- added C55, C56, C57: 100nF/50V, Capacitor_SMD:C_0402_1005Metric, symbol Device:C
- added R57, R58, R59, R60, R61, R62, R63, R64, R65, R66, R67, R68: 1M, Resistor_SMD:R_0402_1005Metric, symbol Device:R
- R41: value 4.7k -> 10k; LCSC C25900 -> C25744; MPN 0402WGF4701TCE -> 0402WGF1002TCE
- R42, R43: value 4.7k -> 100k; LCSC C25900 -> C25741; MPN 0402WGF4701TCE -> 0402WGF1003TCE
- R44: value 10k -> 4.7k; LCSC C25744 -> C25900; MPN 0402WGF1002TCE -> 0402WGF4701TCE
- R45, R46: value 100k -> 4.7k; LCSC C25741 -> C25900; MPN 0402WGF1003TCE -> 0402WGF4701TCE
- R47: value 1M -> 4.7k; LCSC C26083 -> C25900; MPN 0402WGF1004TCE -> 0402WGF4701TCE
- R48: value 1M -> 10k; LCSC C26083 -> C25744; MPN 0402WGF1004TCE -> 0402WGF1002TCE
- R49, R50: value 1M -> 100k; LCSC C26083 -> C25741; MPN 0402WGF1004TCE -> 0402WGF1003TCE
Connections:
- net +3V3: now also C46.1, C48.1, C50.1, R41.2, R46.2, R47.2, C55.1, C56.1; no longer C47.1, C49.1, C53.1, R42.2, R43.2
- net BOOT_B: now also R57.1; no longer R53.1
- net BOOT_DIR: now also R50.1; no longer R46.1
- net GND: now also R42.2, R43.2, R54.2, R55.2, R56.2, U15.10 (A8), C55.2, C56.2, C57.2, R57.2, R61.2, R62.2, R63.2, R64.2, R65.2, R66.2; no longer R44.2, R45.2, R46.2, R47.2
- net I2C_DUT_EN: now also R48.1; no longer R44.1
- net I2C_DUT_SCL_MCU: now also R46.1; no longer R42.1
- net I2C_DUT_SDA_MCU: now also R47.1; no longer R43.1
- net I2C_SCL: now also R44.1
- net I2C_SDA: now also R45.1; no longer R41.1
- net IN1_B: now also R51.1; no longer R47.1
- net IN2_B: now also R52.1; no longer R48.1
- net IN3_B: now also R53.1; no longer R49.1
- net IN4_B: now also R54.1; no longer R50.1
- net LS_OE_N: now also R41.1
- net OUT1_B: now also R61.1
- net OUT2_B: now also R62.1
- net OUT3_B: now also R63.1
- net OUT4_B: now also R64.1
- net RESET_DUT_CTL: now also R49.1; no longer R45.1
- net SPI_CS_B: now also R68.1
- net SPI_MISO_B: now also R55.1; no longer R51.1
- net SPI_MOSI_B: now also R66.1
- net SPI_SCK_B: now also R65.1
- net SWCLK_B: now also R56.1; no longer R52.1
- net SWCLK_DIR: now also R42.1
- net SWDIO_B: now also R60.1; no longer R56.1
- net SWDIO_DIR: now also R43.1
- net SWO_DUT_B: now also R59.1; no longer R55.1
- net UART_RX_B: now also R58.1; no longer R54.1
- net UART_TX_B: now also R67.1
- net VIO: now also C47.1, C49.1, C53.1, R44.2, R45.2, C57.1, R58.2, R59.2, R60.2, R67.2, R68.2; no longer C46.1, C48.1, C50.1, R41.2, R54.2, R55.2, R56.2
- no-connect marks 1 -> 0
Other:
- moved on the sheet: C46, C47, C48, C49, C50, C51, C52, C53, C54, R41, R42, R43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
