File: connectors.kicad_sch (KiCad schematic)
At the start: 36 parts, among them J4 J_PWR, J5 J_DBG, J6 J_BUS, J7 J_UART_ANA, J8 J_IO, U18 TPD4E05U06DQAR, U19 TPD4E05U06DQAR, U20 TPD4E05U06DQAR, U21 TPD4E05U06DQAR, U22 TPD4E05U06DQAR, U23 TPD4E05U06DQAR, U24 TPD4E05U06DQAR, U25 TPD4E05U06DQAR

Commit message: fix: apply schematic review findings (VIO 5V at power-up, push-pull BOOT, input bias, CC ESD)
Co-Authored-By: Claude Opus 5.5 <noreply@anthropic.com>
Parts:
- removed R45, R46, R47, R48, R49, R50, R51, R52, R53, R54, R55, R56: 100R, Resistor_SMD:R_0402_1005Metric, symbol Device:R
- removed U18, U19: TPD4E05U06DQAR, Package_SON:USON-10_2.5x1.0mm_P0.5mm, symbol Power_Protection:TPD4E05U06DQA
- added R64, R65, R66, R67, R68, R69, R70, R71, R72, R73, R74, R75: 100R, Resistor_SMD:R_0402_1005Metric, symbol Device:R
- added U26, U27: TPD4E05U06DQAR, Package_SON:USON-10_2.5x1.0mm_P0.5mm, symbol Power_Protection:TPD4E05U06DQA
Connections:
- net BOOT_OD is gone; now on net SPI_MOSI_B: R63.1
- net 3V3_DUT: now also U27.4 (D2+); no longer U25.4 (D2+)
- net 3V3_SW: now also U27.5 (D2-); no longer U25.5 (D2-)
- net 5V_DUT: now also U27.1 (D1+); no longer U25.1 (D1+)
- net 5V_SW: now also U27.2 (D1-); no longer U25.2 (D1-)
- net AIN1: now also U25.2 (D1-); no longer U23.2 (D1-)
- net AIN2: now also U25.4 (D2+); no longer U23.4 (D2+)
- net AOUT: now also U25.5 (D2-); no longer U23.5 (D2-)
- net BOOT: now also U25.1 (D1+), R75.2; no longer R63.2, U23.1 (D1+)
- net GND: now also U26.3 (GND), U26.8 (GND), U27.3 (GND), U27.8 (GND)
- net I2C_SCL: now also U23.5 (D2-); no longer U21.5 (D2-)
- net I2C_SDA: now also U23.4 (D2+); no longer U21.4 (D2+)
- net IN1: now also U21.1 (D1+), R65.2
- net IN1_B: now also R65.1
- net IN2: now also U21.2 (D1-), R66.2
- net IN2_B: now also R66.1
- net IN3: now also U21.4 (D2+), R67.2
- net IN3_B: now also R67.1
- net IN4: now also U21.5 (D2-), R68.2
- net IN4_B: now also R68.1
- net OUT1: now also R57.2, U20.1 (D1+)
- net OUT1_B: now also R57.1
- net OUT2: now also R58.2, U20.2 (D1-)
- net OUT2_B: now also R58.1
- net OUT3: now also R59.2, U20.4 (D2+)
- net OUT3_B: now also R59.1
- net OUT4: now also R60.2, U20.5 (D2-)
- net OUT4_B: now also R60.1
- net RESET: now also U24.5 (D2-), R74.2; no longer R62.2, U22.5 (D2-)
- net RESET_OD: now also R74.1; no longer R62.1
- net RX: now also U22.2 (D1-), R69.2; no longer R57.2, U20.2 (D1-)
- net SPI_CS: now also U23.2 (D1-), R64.2; no longer U21.2 (D1-)
- net SPI_CS_B: now also R64.1
- net SPI_MISO: now also U23.1 (D1+), R70.2; no longer R58.2, U21.1 (D1+)
- net SPI_MISO_B: now also R70.1; no longer R58.1
- net SPI_MOSI: now also R63.2, U22.5 (D2-); no longer U20.5 (D2-)
- net SPI_SCK: now also R62.2, U22.4 (D2+); no longer U20.4 (D2+)
- net SPI_SCK_B: now also R62.1
- net SWCLK: now also U24.2 (D1-), R72.2; no longer R60.2, U22.2 (D1-)
- net SWCLK_B: now also R72.1; no longer R60.1
- net SWDIO: now also U24.1 (D1+), R73.2; no longer R61.2, U22.1 (D1+)
- net SWDIO_B: now also R73.1; no longer R61.1
- net SWO: now also U24.4 (D2+), R71.2; no longer R59.2, U22.4 (D2+)
- net SWO_DUT_B: now also R71.1; no longer R59.1
- net TX: now also R61.2, U22.1 (D1+); no longer U20.1 (D1+)
- net UART_RX_B: now also R69.1; no longer R57.1
- net UART_TX_B: now also R61.1
- net VIO: now also U26.1 (D1+); no longer U24.1 (D1+)
- new net BOOT_B: R75.1

Commit message: fix: apply schematic review (LQFP-80 MCU, fixed-rail EN, VIO from 5V_DUT, buttons, ESD per header)
- STM32G431MBT6 (LQFP-80): 14 more GPIO; BOOT_DIR off PB4 (JTRST pull-up at reset)
- Fixed DUT rails: EN on PE7/PE8 with pull-up (on by default, firmware can cut)
- TPS2116 VIN1 from current-limited 5V_DUT instead of +5V
- Two user push buttons (TS-1187A) on PD0/PD1, BOOT0 solder jumper
- TVS after the PTC, buck Cin 10uF/25V 0805, 5th VDD decoupling cap
- No floating translator inputs (U15 A8 to GND, 1M bias on U14 B side)
- ESD channels grouped per header; datasheet field falls back to LCSC page
- Decoupling capacitors declare the pin they decouple (validated against nets)

Co-Authored-By: Claude Opus 5.5 <noreply@anthropic.com>
Parts:
- removed R57, R58, R59, R60, R61, R62, R63, R64, R65, R66, R67, R68: 100R, Resistor_SMD:R_0402_1005Metric, symbol Device:R
- added R76, R77, R78, R79, R80, R81, R82, R83, R84, R85, R86, R87: 100R, Resistor_SMD:R_0402_1005Metric, symbol Device:R
- added TP6: 5V_SW, TestPoint:TestPoint_Pad_D1.5mm, symbol Connector:TestPoint
- added TP7: 5V_DUT, TestPoint:TestPoint_Pad_D1.5mm, symbol Connector:TestPoint
- added TP8: 3V3_SW, TestPoint:TestPoint_Pad_D1.5mm, symbol Connector:TestPoint
- added TP9: 3V3_DUT, TestPoint:TestPoint_Pad_D1.5mm, symbol Connector:TestPoint
Connections:
- net 3V3_DUT: now also TP9.1
- net 3V3_SW: now also TP8.1
- net 5V_DUT: now also TP7.1
- net 5V_SW: now also TP6.1
- net AIN1: now also U24.1 (D1+); no longer U25.2 (D1-)
- net AIN2: now also U24.2 (D1-); no longer U25.4 (D2+)
- net AOUT: now also U24.4 (D2+); no longer U25.5 (D2-)
- net BOOT: now also U26.1 (D1+), R87.2; no longer R75.2, U25.1 (D1+)
- net BOOT_B: now also R87.1; no longer R75.1
- net I2C_SCL: now also U22.2 (D1-); no longer U23.5 (D2-)
- net I2C_SDA: now also U22.1 (D1+); no longer U23.4 (D2+)
- net IN1: now also R77.2
- net IN1_B: now also R77.1
- net IN2: now also R78.2
- net IN2_B: now also R78.1
- net IN3: now also R79.2
- net IN3_B: now also R79.1
- net IN4: now also R80.2
- net IN4_B: now also R80.1
- net OUT1: now also R69.2
- net OUT1_B: now also R69.1
- net OUT2: now also R70.2
- net OUT2_B: now also R70.1
- net OUT3: now also R71.2
- net OUT3_B: now also R71.1
- net OUT4: now also R72.2
- net OUT4_B: now also R72.1
- net RESET: now also U25.5 (D2-), R86.2; no longer R74.2, U24.5 (D2-)
- net RESET_OD: now also R86.1; no longer R74.1
- net RX: now also U23.5 (D2-), R81.2; no longer R69.2, U22.2 (D1-)
- net SPI_CS: now also R76.2
- net SPI_CS_B: now also R76.1
- net SPI_MISO: now also R82.2; no longer R70.2
- net SPI_MISO_B: now also R82.1; no longer R70.1
- net SPI_MOSI: now also R75.2
- net SPI_MOSI_B: now also R75.1
- net SPI_SCK: now also R74.2
- net SPI_SCK_B: now also R74.1
- net SWCLK: now also U25.2 (D1-), R84.2; no longer R72.2, U24.2 (D1-)
- net SWCLK_B: now also R84.1; no longer R72.1
- net SWDIO: now also U25.1 (D1+), R85.2; no longer R73.2, U24.1 (D1+)
- net SWDIO_B: now also R85.1; no longer R73.1
- net SWO: now also U25.4 (D2+), R83.2; no longer R71.2, U24.4 (D2+)
- net SWO_DUT_B: now also R83.1; no longer R71.1
- net TX: now also R73.2, U23.4 (D2+); no longer U22.1 (D1+)
- net UART_RX_B: now also R81.1; no longer R69.1
- net UART_TX_B: now also R73.1
- net VIO: now also U26.2 (D1-); no longer U26.1 (D1+)
Other:
- note added: "DUT rail test points"
- moved on the sheet: H1, H2, H3, H4, R69, R70, R71, R72, R73, R74, R75, U22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

Commit message: fix: assign MCU pins to the PCB floor plan, drop test points duplicated by headers
- EN_5V/EN_3V3 on PD8/PD9 and BOOT_DIR on PD10 (pins facing the power and debug blocks)
- BTN1/BTN2 on PE11/PE10 and LED_HB on PE12 (pins facing the top-right corner)
- Second buck output capacitor declared next to the first one
- DUT rail and VIO test points removed: J_PWR / J_DBG pins expose those nets

Co-Authored-By: Claude Opus 5.5 <noreply@anthropic.com>
Parts:
- removed TP6: 5V_SW, TestPoint:TestPoint_Pad_D1.5mm, symbol Connector:TestPoint
- removed TP7: 5V_DUT, TestPoint:TestPoint_Pad_D1.5mm, symbol Connector:TestPoint
- removed TP8: 3V3_SW, TestPoint:TestPoint_Pad_D1.5mm, symbol Connector:TestPoint
- removed TP9: 3V3_DUT, TestPoint:TestPoint_Pad_D1.5mm, symbol Connector:TestPoint
Other:
- note added: "DUT rails and VIO are probed on J_PWR / J_DBG pins (no separate test points)."
- note removed: "DUT rail test points"
- moved on the sheet: H1, H2, H3, H4
