File: vio.kicad_sch (KiCad schematic)
At the start: 16 parts, among them Q1 2N7002, U11 TPS2116DRLR, U12 AP2127K-ADJTRG1

Commit message: fix: apply schematic review findings (VIO 5V at power-up, push-pull BOOT, input bias, CC ESD)
Co-Authored-By: Claude Opus 5.5 <noreply@anthropic.com>
Parts:
- removed U11: TPS2116DRLR, Package_TO_SOT_SMD:SOT-583-8, symbol Power_Management:TPS2116DRL
- removed U12: AP2127K-ADJTRG1, Package_TO_SOT_SMD:SOT-23-5, symbol Regulator_Linear:AP2127K-ADJ
- added R36: 100k, Resistor_SMD:R_0402_1005Metric, symbol Device:R
- added U12: TPS2116DRLR, Package_TO_SOT_SMD:SOT-583-8, symbol Power_Management:TPS2116DRL
- added U13: AP2127K-ADJTRG1, Package_TO_SOT_SMD:SOT-23-5, symbol Regulator_Linear:AP2127K-ADJ
- C39: value 10uF/10V -> 1uF/25V; footprint Capacitor_SMD:C_0603_1608Metric -> Capacitor_SMD:C_0402_1005Metric; LCSC C19702 -> C52923; MPN CL10A106KP8NNNC -> CL05A105KA5NQNC
- R31: value 100k -> 22k; LCSC C25741 -> C25768; MPN 0402WGF1003TCE -> 0402WGF2202TCE
- R32: value 30k -> 100k; LCSC C25776 -> C25741; MPN 0402WGF3002TCE -> 0402WGF1003TCE
- R33: value 24k -> 30k; LCSC C25769 -> C25776; MPN 0402WGF2402TCE -> 0402WGF3002TCE
- R34: value 16k -> 24k; LCSC C25759 -> C25769; MPN 0402WGF1602TCE -> 0402WGF2402TCE
- R35: value 100k -> 16k; LCSC C25741 -> C25759; MPN 0402WGF1003TCE -> 0402WGF1602TCE
Connections:
- net +3V3 is gone; now on net VIO_PR1: R30.2
- net +5V: now also R30.1, U12.3 (VIN1), U13.1 (VIN), U13.3 (EN)
- net GND: now also R32.2, R34.2, R36.2, U12.1 (GND), U13.2 (GND); no longer R33.2, R35.2
- net VIO: now also U12.2 (VOUT), U12.7 (VOUT)
- net VIO_ADJ: now also R33.2, R35.1, U13.4 (ADJ); no longer R32.2, R33.1
- net VIO_LDO: now also R33.1, U12.6 (VIN2), U13.5 (VOUT); no longer R32.1
- net VIO_MODE: now also R32.1, U12.5 (MODE); no longer R31.1
- net VIO_PR1: now also R31.1, U12.4 (PR1); no longer R30.1
- net VIO_VSEL: now also R36.1; no longer R35.1
- net VSEL_D: now also R35.2; no longer R34.2

Commit message: fix: apply schematic review (LQFP-80 MCU, fixed-rail EN, VIO from 5V_DUT, buttons, ESD per header)
- STM32G431MBT6 (LQFP-80): 14 more GPIO; BOOT_DIR off PB4 (JTRST pull-up at reset)
- Fixed DUT rails: EN on PE7/PE8 with pull-up (on by default, firmware can cut)
- TPS2116 VIN1 from current-limited 5V_DUT instead of +5V
- Two user push buttons (TS-1187A) on PD0/PD1, BOOT0 solder jumper
- TVS after the PTC, buck Cin 10uF/25V 0805, 5th VDD decoupling cap
- No floating translator inputs (U15 A8 to GND, 1M bias on U14 B side)
- ESD channels grouped per header; datasheet field falls back to LCSC page
- Decoupling capacitors declare the pin they decouple (validated against nets)

Co-Authored-By: Claude Opus 5.5 <noreply@anthropic.com>
Parts:
- removed C37, C38, C39: 1uF/25V, Capacitor_SMD:C_0402_1005Metric, symbol Device:C
- removed R30: 10k, Resistor_SMD:R_0402_1005Metric, symbol Device:R
- removed R31: 22k, Resistor_SMD:R_0402_1005Metric, symbol Device:R
- removed R32: 100k, Resistor_SMD:R_0402_1005Metric, symbol Device:R
- removed R33: 30k, Resistor_SMD:R_0402_1005Metric, symbol Device:R
- removed TP10: VIO, TestPoint:TestPoint_Pad_D1.5mm, symbol Connector:TestPoint
- added C43, C44: 1uF/25V, Capacitor_SMD:C_0402_1005Metric, symbol Device:C
- added C45: 1nF/50V, Capacitor_SMD:C_0402_1005Metric, symbol Device:C
- added R37: 30k, Resistor_SMD:R_0402_1005Metric, symbol Device:R
- added R38: 24k, Resistor_SMD:R_0402_1005Metric, symbol Device:R
- added R39: 16k, Resistor_SMD:R_0402_1005Metric, symbol Device:R
- added R40: 100k, Resistor_SMD:R_0402_1005Metric, symbol Device:R
- added TP5: VIO, TestPoint:TestPoint_Pad_D1.5mm, symbol Connector:TestPoint
- C42: value 1nF/50V -> 1uF/25V; LCSC C1523 -> C52923; MPN 0402B102K500NT -> CL05A105KA5NQNC; Manufacturer FH -> Samsung
- R34: value 24k -> 10k; LCSC C25769 -> C25744; MPN 0402WGF2402TCE -> 0402WGF1002TCE
- R35: value 16k -> 22k; LCSC C25759 -> C25768; MPN 0402WGF1602TCE -> 0402WGF2202TCE
Connections:
- net +5V: now also R34.1, C43.1; no longer C40.1, U12.3 (VIN1)
- net GND: now also C42.2, R35.2, C43.2, C44.2, R38.2, R40.2; no longer R34.2
- net VIO: now also C42.1, TP5.1
- net VIO_ADJ: now also C45.2, R37.2, R38.1, R39.1; no longer C42.2, R34.1, R35.1
- net VIO_LDO: now also C44.1, C45.1, R37.1; no longer C42.1
- net VIO_MODE: now also R36.1
- net VIO_PR1: now also R34.2, R35.1
- net VIO_VSEL: now also R40.1; no longer R36.1
- net VSEL_D: now also R39.2; no longer R35.2
- new net 5V_DUT: C40.1, U12.3 (VIN1)
Other:
- note added: "TPS2116: MODE=1 PR1=1 -> 5V_DUT ; MODE=1 PR1=0 -> LDO ; MODE=0 PR1=1 -> off (external VIO from J_PWR/J_DBG). MODE=0 PR1=0 is forbidden (selects 5 V)."
- note removed: "TPS2116: MODE=1 PR1=1 -> 5V_SYS ; MODE=1 PR1=0 -> LDO ; MODE=0 PR1=1 -> off (external VIO from J_PWR/J_DBG). MODE=0 PR1=0 is forbidden (selects 5 V)."
- moved on the sheet: C40, C41, C42, R34, R35, R36

Commit message: fix: assign MCU pins to the PCB floor plan, drop test points duplicated by headers
- EN_5V/EN_3V3 on PD8/PD9 and BOOT_DIR on PD10 (pins facing the power and debug blocks)
- BTN1/BTN2 on PE11/PE10 and LED_HB on PE12 (pins facing the top-right corner)
- Second buck output capacitor declared next to the first one
- DUT rail and VIO test points removed: J_PWR / J_DBG pins expose those nets

Co-Authored-By: Claude Opus 5.5 <noreply@anthropic.com>
Parts:
- removed TP5: VIO, TestPoint:TestPoint_Pad_D1.5mm, symbol Connector:TestPoint
