File: OOTY.kicad_sch (KiCad schematic)
At the start: 0 parts

Commit message: feat: generate hierarchical schematic (power, mcu, sensing, vio, translators, connectors)
Co-Authored-By: Claude Opus 5.5 <noreply@anthropic.com>
Other:
- added sheet connectors (connectors.kicad_sch)
- added sheet mcu (mcu.kicad_sch)
- added sheet power (power.kicad_sch)
- added sheet sensing (sensing.kicad_sch)
- added sheet translators (translators.kicad_sch)
- added sheet vio (vio.kicad_sch)
- note added: "OOTY rev A - hierarchical schematic generated by scripts/build_schematic.py"
- note added: "Specification: SPEC.md - design notes and calculations: NOTES.md"
- company: (none) -> OOTY
- title: (none) -> OOTY - USB Hardware-in-the-Loop board

Commit message: feat: dual-range current sensing and fixed-rail readback in the schematic (TASK-011)
New sheets range_5v_sw, range_3v3_sw and readback appended at the end of the
hierarchy (existing references unchanged). Shunts now end on *_MID, INA226
Vin- on *_MID, MCU pins remapped per NOTES.md. ERC 0 errors, netlist and BOM
0 mismatches.

Co-Authored-By: Claude Opus 5.5 <noreply@anthropic.com>
Other:
- added sheet range_3v3_sw (range_3v3_sw.kicad_sch)
- added sheet range_5v_sw (range_5v_sw.kicad_sch)
- added sheet readback (readback.kicad_sch)
Changed lines of the file:
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@@
+	)
+	(sheet
+		(at 220.5 80.64)
+		(size 50.8 20.32)
+		(exclude_from_sim no)
+		(in_bom yes)
+		(on_board yes)
+		(dnp no)
+		(fields_autoplaced yes)
+		(stroke
+			(width 0.1524)
+			(type solid)
+		)
+		(fill
+			(color 0 0 0 0)
+		)
+		(property "Sheetname" "range_3v3_sw"
+			(at 220.5 80.01 0)
+			(show_name no)
+			(do_not_autoplace no)
+			(effects
+				(font
+					(size 1.27 1.27)
+				)
+				(justify left bottom)
+			)
+		)
+		(property "Sheetfile" "range_3v3_sw.kicad_sch"
+			(at 220.5 101.6 0)
+			(show_name no)
+			(do_not_autoplace no)
+			(effects
+				(font
+					(size 1.27 1.27)
+				)
+				(justify left top)
+			)
+		)
+		(instances
+			(project "OOTY"
+				(path "/896c938c-ef54-5782-bb20-81d92df4de86"
+					(page "9")
+				)
+			)
+		)
 	)
 	(sheet
@@
 				)
 			)
+		)
+	)
+	(sheet
+		(at 157 80.64)
+		(size 50.8 20.32)
+		(exclude_from_sim no)
+		(in_bom yes)
+		(on_board yes)
+		(dnp no)
+		(fields_autoplaced yes)
+		(stroke
+			(width 0.1524)
+			(type solid)
+		)
+		(fill
+			(color 0 0 0 0)
+		)
+		(property "Sheetname" "range_5v_sw"
+			(at 157 80.01 0)
+			(show_name no)
+			(do_not_autoplace no)
+			(effects
+				(font
+					(size 1.27 1.27)
+				)
+				(justify left bottom)
+			)
+		)
+		(property "Sheetfile" "range_5v_sw.kicad_sch"
+			(at 157 101.6 0)
+			(show_name no)
+			(do_not_autoplace no)
+			(effects
+				(font
+					(size 1.27 1.27)
+				)
+				(justify left top)
+			)
+		)
+		(instances
+			(project "OOTY"
+				(path "/896c938c-ef54-5782-bb20-81d92df4de86"
+					(page "8")
+				)
+			)
+		)
+	)
+	(sheet
+		(at 30 121.28)
+		(size 50.8 20.32)
+		(exclude_from_sim no)
+		(in_bom yes)
+		(on_board yes)
+		(dnp no)
+		(fields_autoplaced yes)
+		(stroke
+			(width 0.1524)
+			(type solid)
+		)
+		(fill
+			(color 0 0 0 0)
+		)
+		(property "Sheetname" "readback"
+			(at 30 120.65 0)
+			(show_name no)
+			(do_not_autoplace no)
+			(effects
+				(font
+					(size 1.27 1.27)
+				)
+				(justify left bottom)
+			)
+		)
+		(property "Sheetfile" "readback.kicad_sch"
+			(at 30 142.24 0)
+			(show_name no)
+			(do_not_autoplace no)
+			(effects
+				(font
+					(size 1.27 1.27)
+				)
+				(justify left top)
+			)
+		)
+		(instances
+			(project "OOTY"
+				(path "/896c938c-ef54-5782-bb20-81d92df4de86"
+					(page "10")
+				)
+			)
