File: range_3v3_sw.kicad_sch (KiCad schematic)
At the start: 28 parts, among them Q5 AO3401A, Q6 2N7002, U32 TLV7021DBVR, U33 SN74LVC1G74DCUR, U34 INA190A2IDCKR, U35 INA190A2IDCKR

Commit message: fix: schematic review of TASK-011 (DNP cap part number, parallel-path note, UCPD/PB4 note)
Co-Authored-By: Claude Opus 5.5 <noreply@anthropic.com>
Parts:
- C65: value 1uF DNP -> 1uF/25V X7R; LCSC_DNP (none) -> C29936; MPN (none) -> CL10B105KA8NNNC; Manufacturer (none) -> Samsung
Other:
- note added: "100R, JP (BYPASS), M7 and AO3401A are in parallel between *_MID and the rail output."
Changed lines of the file:
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@@
 		)
 	)
-	(text "M7: clamps the drop while the range switches. JP open: bridge it to bypass the 100R."
+	(text "100R, JP (BYPASS), M7 and AO3401A are in parallel between *_MID and the rail output."
 		(exclude_from_sim no)
 		(at 20 265.43 0)
@@
 		)
 	)
+	(text "M7: clamps the drop while the range switches. JP open: bridge it to bypass the 100R."
+		(exclude_from_sim no)
+		(at 20 270.51 0)
+		(effects
+			(font
+				(size 1.27 1.27)
+			)
+			(justify left bottom)
+		)
+	)
 	(text "3V3_SW amplifiers (x50)"
 		(exclude_from_sim no)
@@
 			)
 		)
-		(property "Value" "1uF DNP"
+		(property "Value" "1uF/25V X7R"
 			(at 38.1 171.45 90)
 			(show_name no)
@@
 			)
 		)
-		(property "Datasheet" ""
+		(property "Datasheet" "https://www.lcsc.com/product-detail/C29936.html"
 			(at 38.1 167.64 0)
 			(hide yes)
@@
 			(at 38.1 167.64 0)
 			(hide yes)
+			(show_name no)
+			(do_not_autoplace no)
+			(effects
+				(font
+					(size 1.27 1.27)
+				)
+			)
+		)
+		(property "MPN" "CL10B105KA8NNNC"
+			(at 38.1 167.64 0)
+			(hide yes)
+			(show_name no)
+			(do_not_autoplace no)
+			(effects
+				(font
+					(size 1.27 1.27)
+				)
+			)
+		)
+		(property "Manufacturer" "Samsung"
+			(at 38.1 167.64 0)
+			(hide yes)
+			(show_name no)
+			(do_not_autoplace no)
+			(effects
+				(font
+					(size 1.27 1.27)
+				)
+			)
+		)
+		(property "LCSC_DNP" "C29936"
+			(at 38.1 167.64 0)
+			(hide yes)
