File: range_5v_sw.kicad_sch (KiCad schematic)
At the start: 28 parts, among them Q3 AO3401A, Q4 2N7002, U28 TLV7021DBVR, U29 SN74LVC1G74DCUR, U30 INA190A2IDCKR, U31 INA190A2IDCKR

Commit message: fix: schematic review of TASK-011 (DNP cap part number, parallel-path note, UCPD/PB4 note)
Co-Authored-By: Claude Opus 5.5 <noreply@anthropic.com>
Parts:
- C58: value 1uF DNP -> 1uF/25V X7R; LCSC_DNP (none) -> C29936; MPN (none) -> CL10B105KA8NNNC; Manufacturer (none) -> Samsung
Other:
- note added: "100R, JP (BYPASS), M7 and AO3401A are in parallel between *_MID and the rail output."
Changed lines of the file:
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@@
 	(text "M7: clamps the drop while the range switches. JP open: bridge it to bypass the 100R."
 		(exclude_from_sim no)
+		(at 20 270.51 0)
+		(effects
+			(font
+				(size 1.27 1.27)
+			)
+			(justify left bottom)
+		)
+	)
+	(text "100R, JP (BYPASS), M7 and AO3401A are in parallel between *_MID and the rail output."
+		(exclude_from_sim no)
 		(at 20 265.43 0)
 		(effects
@@
 			)
 		)
-		(property "Value" "1uF DNP"
+		(property "Value" "1uF/25V X7R"
 			(at 36.83 167.64 90)
 			(show_name no)
@@
 			)
 		)
-		(property "Datasheet" ""
+		(property "Datasheet" "https://www.lcsc.com/product-detail/C29936.html"
 			(at 36.83 163.83 0)
 			(hide yes)
@@
 			(at 36.83 163.83 0)
 			(hide yes)
+			(show_name no)
+			(do_not_autoplace no)
+			(effects
+				(font
+					(size 1.27 1.27)
+				)
+			)
+		)
+		(property "MPN" "CL10B105KA8NNNC"
+			(at 36.83 163.83 0)
+			(hide yes)
+			(show_name no)
+			(do_not_autoplace no)
+			(effects
+				(font
+					(size 1.27 1.27)
+				)
+			)
+		)
+		(property "Manufacturer" "Samsung"
+			(at 36.83 163.83 0)
+			(hide yes)
+			(show_name no)
+			(do_not_autoplace no)
+			(effects
+				(font
+					(size 1.27 1.27)
+				)
+			)
+		)
+		(property "LCSC_DNP" "C29936"
+			(at 36.83 163.83 0)
+			(hide yes)
